Commit message: Added collision elements to URDF

File: dobot_e6_description/urdf/mech/base_link.urdf.xacro (robot description, xacro)
@@ -10,7 +10,7 @@
             </visual>
             <collision>
-                <origin xyz="0 0 0.01749" rpy="0 0 0"/>
+                <origin xyz="0 -0.02087 0.00185" rpy="0 0 0"/>
                 <geometry>
-                    <box size="0.150 0.2 0.0"/>
+                    <box size="0.140 0.2 0.1077"/>
                 </geometry>
             </collision>
@@ -18,5 +18,4 @@
                 <!-- TODO-->
                 <!-- Based on the actual mass we need to update the inertial section-->
-                <!-- stl frame/link frame is equal to the COM (defined in CAD) therefore, origin is a zero vector-->
                 <mass value="1.0" />
                 <origin xyz="0 0 0" rpy="0 0 0"/>

File: dobot_e6_description/urdf/mech/dobot_e6_arm.urdf.xacro (robot description, xacro)
@@ -34,7 +34,7 @@
             </visual>
             <collision>
-                <origin xyz="0 0 0" rpy="0 0 0" />
+                <origin xyz="0 0.01025 -0.00145" rpy="0 0 0" />
                 <geometry>
-                    <box size="0 0 0"/>
+                    <box size="0.100 0.090 0.085"/>
                 </geometry>
             </collision>
@@ -51,7 +51,7 @@
             </visual>
             <collision>
-                <origin xyz="0 0 0" rpy="0 0 0" />
+                <origin xyz="0 -0.09375 0.00283" rpy="0 0 0" />
                 <geometry>
-                    <box size="0 0 0"/>
+                    <box size="0.080 0.267 0.080"/>
                 </geometry>
             </collision>
@@ -60,5 +60,5 @@
             <!-- TODO: Fix inertial-->
              <!-- TODO: Fix inertial origin-->
-            <xacro:link_inertial mass="${link2_mass}" ixx="0.000148" iyy="0.000148" izz="0.000096"/>
+            <xacro:link_inertial mass="${link3_mass}" ixx="0.000148" iyy="0.000148" izz="0.000096"/>
             <visual>
                 <origin xyz="0 0 0" rpy="0 0 0" />
@@ -68,7 +68,7 @@
             </visual>
             <collision>
-                <origin xyz="0 0 0" rpy="0 0 0" />
+                <origin xyz="0 -0.080 0.00283" rpy="0 0 0" />
                 <geometry>
-                    <box size="0 0 0"/>
+                    <box size="0.080 0.230 0.080"/>
                 </geometry>
             </collision>
@@ -77,5 +77,5 @@
             <!-- TODO: Fix inertial-->
              <!-- TODO: Fix inertial origin-->
-            <xacro:link_inertial mass="${link2_mass}" ixx="0.000148" iyy="0.000148" izz="0.000096"/>
+            <xacro:link_inertial mass="${link4_mass}" ixx="0.000148" iyy="0.000148" izz="0.000096"/>
             <visual>
                 <origin xyz="0 0 0" rpy="0 0 0" />
@@ -85,7 +85,7 @@
             </visual>
             <collision>
-                <origin xyz="0 0 0" rpy="0 0 0" />
+                <origin xyz="0 -0.0085 -0.0055" rpy="0 0 0" />
                 <geometry>
-                    <box size="0 0 0"/>
+                    <box size="0.065 0.087 0.077"/>
                 </geometry>
             </collision>
@@ -94,5 +94,5 @@
             <!-- TODO: Fix inertial-->
              <!-- TODO: Fix inertial origin-->
-            <xacro:link_inertial mass="${link2_mass}" ixx="0.000148" iyy="0.000148" izz="0.000096"/>
+            <xacro:link_inertial mass="${link5_mass}" ixx="0.000148" iyy="0.000148" izz="0.000096"/>
             <visual>
                 <origin xyz="0 0 0" rpy="0 0 0" />
@@ -102,7 +102,7 @@
             </visual>
             <collision>
-                <origin xyz="0 0 0" rpy="0 0 0" />
+                <origin xyz="0 0.00965 -0.00825" rpy="0 0 0" />
                 <geometry>
-                    <box size="0 0 0"/>
+                    <box size="0.065 0.109 0.0815"/>
                 </geometry>
             </collision>
@@ -111,5 +111,5 @@
             <!-- TODO: Fix inertial-->
              <!-- TODO: Fix inertial origin-->
-            <xacro:link_inertial mass="${link2_mass}" ixx="0.000148" iyy="0.000148" izz="0.000096"/>
+            <xacro:link_inertial mass="${flange_mass}" ixx="0.000148" iyy="0.000148" izz="0.000096"/>
             <visual>
                 <origin xyz="0 0 0" rpy="0 0 0" />
@@ -121,5 +121,5 @@
                 <origin xyz="0 0 0" rpy="0 0 0" />
                 <geometry>
-                    <box size="0 0 0"/>
+                    <cylinder radius="0.0400" length="0.021"/>
                 </geometry>
             </collision>
@@ -163,5 +163,6 @@
             <parent link="${prefix}link5" />
             <child link="${prefix}flange" />
-            <origin xyz="-0.00362 -0.05989 0" rpy="${pi/2} 0 0" />
+            <!--origin xyz="-0.00362 -0.05989 0" rpy="${pi/2} 0 0" /-->
+            <origin xyz="0 -0.05989 0" rpy="${pi/2} 0 0" />
             <axis xyz="0 0 1" />
             <limit effort="${joint_effort}" lower="-2.879793" upper="2.879793" velocity="${joint_velocity}"/>
