Commit message: Modified urdf files

File: dobot_e6_description/urdf/mech/dobot_e6_arm.urdf.xacro (robot description, xacro)
@@ -128,5 +128,5 @@
             <parent link="${prefix}base_link" />
             <child link="${prefix}link1" />
-            <origin xyz="0.00093 0.02088 0.11484" rpy="0 0 0" />
+            <origin xyz="0 0 0.0967" rpy="0 0 0" />
             <axis xyz="0 0 1" />
             <limit effort="${joint_effort}" lower="-2.879793" upper="2.879793" velocity="${joint_velocity}"/>
@@ -135,5 +135,5 @@
             <parent link="${prefix}link1" />
             <child link="${prefix}link2" />
-            <origin xyz="0.00586 0.09699 0" rpy="${-pi/2} 0 0" />
+            <origin xyz="0 0.09717 0" rpy="${-pi/2} 0 0" />
             <axis xyz="0 0 1" />
             <limit effort="${joint_effort}" lower="-2.879793" upper="2.879793" velocity="${joint_velocity}"/>
@@ -142,5 +142,5 @@
             <parent link="${prefix}link2" />
             <child link="${prefix}link3" />
-            <origin xyz="-0.00476 -0.189 -0.07874" rpy="0 ${pi} 0" />
+            <origin xyz="0 -0.189 -0.07888" rpy="0 ${pi} 0" />
             <axis xyz="0 0 1" />
             <limit effort="${joint_effort}" lower="-2.879793" upper="2.879793" velocity="${joint_velocity}"/>
@@ -149,5 +149,5 @@
             <parent link="${prefix}link3" />
             <child link="${prefix}link4" />
-            <origin xyz="0.00520 -0.160 -0.08606" rpy="0 ${pi} 0" />
+            <origin xyz="0 -0.160 -0.08621" rpy="0 ${pi} 0" />
             <axis xyz="0 0 1" />
             <limit effort="${joint_effort}" lower="-2.879793" upper="2.879793" velocity="${joint_velocity}"/>

Commit message: Fixed zero position with luka

File: dobot_e6_description/urdf/mech/dobot_e6_arm.urdf.xacro (robot description, xacro)
@@ -128,5 +128,5 @@
             <parent link="${prefix}base_link" />
             <child link="${prefix}link1" />
-            <origin xyz="0 0 0.0967" rpy="0 0 0" />
+            <origin xyz="0 0 0.0967" rpy="0 0 ${pi}" />
             <axis xyz="0 0 1" />
             <limit effort="${joint_effort}" lower="-2.879793" upper="2.879793" velocity="${joint_velocity}"/>
