Commit message: made some fixes to urdf

File: dobot_e6_description/urdf/mech/tester_end_effector.urdf.xacro (robot description, xacro)
@@ -6,5 +6,5 @@
                 <origin xyz="0.0 0.0 0.04"/>
                 <mass value="0.15"/>
-                <inertia ixx="0.0" ixy="0.0" ixz="0.0" iyy="0.0" iyz="0.0" izz="0.0"/>
+                <inertia ixx="1e-5" ixy="0.0" ixz="0.0" iyy="1e-5" iyz="0.0" izz="1e-5"/>
             </inertial>
             <visual>

File: dobot_e6_description/urdf/robots/dobot_e6.urdf.xacro (robot description, xacro)
@@ -1,5 +1,5 @@
 <?xml version="1.0"?>
 <robot xmlns:xacro="http://www.ros.org/wiki/xacro" name="me6_robot">
-    <xacro:arg name="use_tester_end_effector" default="false"/>
+    <xacro:arg name="use_tester_end_effector" default="true"/>
     <xacro:arg name="robot_name" default="me6_robot"/>
     <xacro:arg name='use_mock_hardware' default='true'/>

Commit message: Added TCP for testing gripper, will manually modify config files for moveit

File: dobot_e6_description/urdf/mech/tester_end_effector.urdf.xacro (robot description, xacro)
@@ -21,4 +21,5 @@
             </collision>
         </link>
+        <link name="dummy_end_effector"/>
         <joint name="joint_end_effector" type="fixed">
             <origin xyz="0.0 0.0 0.021"/>
@@ -26,4 +27,9 @@
             <child link="tester_link"/>
         </joint>
+        <joint name="joint_dummy_end_effector" type="fixed">
+            <origin xyz="0.0 0.0 0.160"/>
+            <parent link="tester_link"/>
+            <child link="dummy_end_effector"/>
+        </joint>
     </xacro:macro>
 </robot>
