Commit message: Scalled collision STLs

File: dobot_e6_description/urdf/mech/weed_removal_tool.urdf.xacro (robot description, xacro)
@@ -20,5 +20,5 @@
                 <origin xyz="0.0 0.0 0.0" rpy="0.0 0.0 0.0"/>
                 <geometry>
-                    <mesh filename="file://$(find dobot_e6_description)/meshes/weed_removal_tool/visual/gripper_housing.STL" />
+                    <mesh filename="file://$(find dobot_e6_description)/meshes/weed_removal_tool/visual/gripper_housing.STL" scale="1.05 1.05 1.05"/>
                 </geometry>
             </collision>
@@ -42,5 +42,5 @@
                 <origin xyz="0.0 0.0 0.0" rpy="0.0 0.0 0.0"/>
                 <geometry>
-                    <mesh filename="file://$(find dobot_e6_description)/meshes/weed_removal_tool/visual/blade_left.STL" />
+                    <mesh filename="file://$(find dobot_e6_description)/meshes/weed_removal_tool/visual/blade_left.STL" scale="1.05 1.05 1.05"/>
                 </geometry>
             </collision>
@@ -64,5 +64,5 @@
                 <origin xyz="0.0 0.0 0.0" rpy="0.0 0.0 0.0"/>
                 <geometry>
-                    <mesh filename="file://$(find dobot_e6_description)/meshes/weed_removal_tool/visual/blade_right.STL" />
+                    <mesh filename="file://$(find dobot_e6_description)/meshes/weed_removal_tool/visual/blade_right.STL" scale="1.05 1.05 1.05"/>
                 </geometry>
             </collision>
