Commit message: Added world frame

File: dobot_e6_description/urdf/robots/dobot_e6.urdf.xacro (robot description, xacro)
@@ -10,5 +10,6 @@
           <parent link="world"/>
           <child link="base_link"/>
-          <origin xyz="0 0 0.03886" rpy="0 0 0"/>
+          <!--origin xyz="0 0 0.03886" rpy="0 0 0"/-->
+          <origin xyz="0.062 0.0863 0.052" rpy="0 0 0"/>
       </joint>
     </xacro:if>

Commit message: added req files for launching framework with gripper plugin

File: dobot_e6_description/urdf/robots/dobot_e6.urdf.xacro (robot description, xacro)
@@ -5,8 +5,10 @@
     <xacro:arg name="robot_name" default="me6_robot"/>
     <xacro:arg name='use_mock_hardware' default='false'/>
+    <xacro:arg name='use_gripper_hardware_interface' default='true'/>
     <xacro:include filename="$(find dobot_e6_description)/urdf/mech/dobot_e6_arm.urdf.xacro"/>
     <xacro:include filename="$(find dobot_e6_description)/urdf/mech/tester_end_effector.urdf.xacro"/>
     <xacro:include filename="$(find dobot_e6_description)/urdf/mech/weed_removal_tool.urdf.xacro"/>
     <xacro:include filename="$(find dobot_e6_description)/urdf/control/dobot_e6_ros2_control.urdf.xacro"/>
+    <xacro:include filename="$(find dobot_e6_description)/urdf/control/gripper_control.urdf.xacro"/>
     <xacro:dobot_e6_arm/>
     <!-- if argument for test end_effector-->
@@ -20,5 +22,6 @@
         <xacro:weed_removal_tool/>
     </xacro:if>
-    <!--xacro:dobot_e6_ros2_control
-        use_mock_hardware="$(arg use_mock_hardware)"/-->
+    <xacro:if value="$(arg use_gripper_hardware_interface)">
+        <xacro:gripper_ros2_control/>
+    </xacro:if>
 </robot>

File: me6_moveit/config/me6_robot.ros2_control.xacro (robot description, xacro)
@@ -50,5 +50,5 @@
                 <state_interface name="velocity"/>
             </joint>
-            <joint name="gripper_controller">
+            <!--joint name="gripper_controller">
                 <command_interface name="position"/>
                 <state_interface name="position">
@@ -56,5 +56,5 @@
                 </state_interface>
                 <state_interface name="velocity"/>
-            </joint>
+            </joint-->
         </ros2_control>
     </xacro:macro>

File: me6_moveit/config/me6_robot.urdf.xacro (robot description, xacro)
@@ -6,4 +6,4 @@
     <!-- Import control_xacro -->
     <xacro:include filename="me6_robot.ros2_control.xacro" />
-    <xacro:me6_robot_ros2_control name="FakeSystem" initial_positions_file="$(arg initial_positions_file)"/>
+    <!--xacro:me6_robot_ros2_control name="FakeSystem" initial_positions_file="$(arg initial_positions_file)"/-->
 </robot>
