Commit message: Updated moveit config files for weed gripper

File: me6_moveit/config/me6_robot.ros2_control.xacro (robot description, xacro)
@@ -2,5 +2,5 @@
 <robot xmlns:xacro="http://www.ros.org/wiki/xacro">
     <xacro:macro name="me6_robot_ros2_control" params="name initial_positions_file">
-        <xacro:property name="initial_positions" value="${load_yaml(initial_positions_file)['initial_positions']}"/>
+        <xacro:property name="initial_positions" value="${xacro.load_yaml(initial_positions_file)['initial_positions']}"/>
         <ros2_control name="${name}" type="system">
             <hardware>
@@ -50,4 +50,11 @@
                 <state_interface name="velocity"/>
             </joint>
+            <joint name="gripper_controller">
+                <command_interface name="position"/>
+                <state_interface name="position">
+                  <param name="initial_value">${initial_positions['gripper_controller']}</param>
+                </state_interface>
+                <state_interface name="velocity"/>
+            </joint>
         </ros2_control>
     </xacro:macro>

File: me6_moveit/config/me6_robot.urdf.xacro (robot description, xacro)
@@ -3,5 +3,4 @@
     <xacro:arg name="initial_positions_file" default="initial_positions.yaml" />
     <!-- Import me6_robot urdf file -->
-    <!--xacro:include filename="$(find dobot_rviz)/urdf/me6_robot.urdf" /-->
     <xacro:include filename="$(find dobot_e6_description)/urdf/robots/dobot_e6.urdf.xacro" />
     <!-- Import control_xacro -->

Commit message: Added functionality for switching between sim and real, needs testing

File: me6_moveit/config/me6_robot.ros2_control.xacro (robot description, xacro)
@@ -50,5 +50,5 @@
                 <state_interface name="velocity"/>
             </joint>
-            <!--joint name="gripper_controller">
+            <joint name="gripper_controller">
                 <command_interface name="position"/>
                 <state_interface name="position">
@@ -56,5 +56,5 @@
                 </state_interface>
                 <state_interface name="velocity"/>
-            </joint-->
+            </joint>
         </ros2_control>
     </xacro:macro>

File: me6_moveit/config/me6_robot.urdf.xacro (robot description, xacro)
@@ -2,8 +2,21 @@
 <robot xmlns:xacro="http://www.ros.org/wiki/xacro" name="me6_robot">
     <xacro:arg name="initial_positions_file" default="initial_positions.yaml" />
+    <xacro:arg name='use_real_hardware' default='false'/>
+    <xacro:include filename="$(find dobot_e6_description)/urdf/mech/dobot_e6_arm.urdf.xacro"/>
+    <xacro:include filename="$(find dobot_e6_description)/urdf/mech/weed_removal_tool.urdf.xacro"/>
+    <xacro:include filename="$(find dobot_e6_description)/urdf/control/gripper_control.urdf.xacro"/>
+    <xacro:include filename="me6_robot.ros2_control.xacro" />
+    <xacro:dobot_e6_arm/>
+    <xacro:weed_removal_tool/>
+    <xacro:if value="$(arg use_real_hardware)">
+        <xacro:gripper_ros2_control/>
+    </xacro:if>
+    <xacro:unless value="$(arg use_real_hardware)">
+        <xacro:me6_robot_ros2_control name="FakeSystem" initial_positions_file="$(arg initial_positions_file)"/>
+    </xacro:unless>
     <!-- Import me6_robot urdf file -->
-    <xacro:include filename="$(find dobot_e6_description)/urdf/robots/dobot_e6.urdf.xacro" />
+    <!--xacro:include filename="$(find dobot_e6_description)/urdf/robots/dobot_e6.urdf.xacro" /-->
     <!-- Import control_xacro -->
-    <xacro:include filename="me6_robot.ros2_control.xacro" />
+    <!--xacro:include filename="me6_robot.ros2_control.xacro" /-->
     <!--xacro:me6_robot_ros2_control name="FakeSystem" initial_positions_file="$(arg initial_positions_file)"/-->
 </robot>
